File: case/gameboyzero-case.brd (EAGLE design)
At the start: 322 x 192 mm, 0 parts

Commit message: New Silk and New Case files
Other:
- board size 322 x 192 mm -> 239 x 201 mm
- board text added: "BATTERY"
- board text added: "BOTTOM"
- board text added: "PI ZERO"
- board text added: "SCREEN"
- board text added: "TOP"
- board text removed: "BOTTOM 1 - A"
- board text removed: "BOTTOM 1 - B"
- board text removed: "BOTTOM 2"
- board text removed: "BOTTOM 3"
- board text removed: "TOP 1"
- board text removed: "TOP 2 - A"
- board text removed: "TOP 2 - B"
