File: case/gameboyzero.brd (EAGLE design)
At the start: 239 x 201 mm, 0 parts

Commit message: Mon 30 Oct 2017 11:48:34 EDT - new case
Parts:
- added H1, H10, H16, H17, H19, H2, H20, H23, H24, H3, H4, H5, H6, H7, H8, H9: MOUNT-HOLE2.8, holes:2,8
Other:
- board size 239 x 201 mm -> 237 x 216 mm
- board text removed: "BATTERY"
- board text removed: "BOTTOM"
- board text removed: "PI ZERO"
- board text removed: "SCREEN"
- board text removed: "TOP"
