File: case/gameboyzero.brd (EAGLE design)
At the start: 337.8 x 172 mm, 32 parts

Commit message: Tue 31 Oct 2017 16:24:41 EDT
Parts:
- added H100, H101, H102, H103, H104, H105, H106, H107, H108, H109, H110, H111, H112, H113, H114, H115, H116, H117, H118, H119, H120, H121, H122, H123, H124, H125, H126, H127, H128, H129, H130, H131, H132, H133, H134, H135, H136, H137, H138, H139, H140, H141, H142, H143, H144, H145, H146, H147, H148, H149, H150, H151, H152, H153, H154, H155, H156, H157, H158, H159, H160, H161, H162, H163, H164, H165, H166, H167, H168, H169, H170, H171, H172, H173, H174, H175, H176, H177, H178, H179, H180, H181, H182, H183, H184, H185, H186, H187, H188, H189, H190, H191, H192, H193, H194, H195, H196, H197, H198, H199, H200, H201, H202, H203, H204, H205, H206, H207, H208, H209, H210, H211, H212, H213, H214, H215, H216, H217, H218, H219, H220, H221, H222, H223, H224, H225, H226, H227, H33, H34, H35, H36, H37, H38, H39, H40, H41, H42, H43, H44, H45, H46, H47, H48, H49, H50, H51, H52, H53, H54, H55, H56, H57, H58, H59, H60, H61, H62, H63, H64, H65, H66, H67, H68, H69, H70, H71, H72, H73, H74, H75, H76, H77, H78, H79, H80, H81, H82, H83, H84, H85, H86, H87, H88, H89, H90, H91, H92, H93, H94, H95, H96, H97, H98, H99: MOUNT-HOLE2.8, holes:2,8
- moved H30 201.5 mm to (83.3, 79.3)
- moved H27 168.8 mm to (83.3, 10.3)
- moved H28 168.8 mm to (146.3, 10.3)
- moved H32 167.5 mm to (229.3, 10.3)
- moved H11 147.3 mm to (83.3, 136.3)
- moved H12 147.3 mm to (146.3, 136.3)
- moved H13 147.3 mm to (146.3, 166.3)
- moved H16 147.2 mm to (156.3, 175.3)
- moved H17 147.2 mm to (219.3, 175.3)
- moved H14 121.1 mm to (83.3, 175.3)
- moved H15 121.1 mm to (146.3, 175.3)
- moved H31 116.0 mm to (146.3, 79.3)
- moved H23 95.7 mm to (156.3, 117.1)
- moved H24 95.7 mm to (219.3, 117.1)
- moved H19 95.2 mm to (156.3, 58.4)
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Other:
- board size 337.8 x 172 mm -> 702.4 x 426.4 mm

Commit message: Tue  7 Nov 2017 15:28:11 EST
Parts:
- removed H1, H10, H100, H101, H102, H103, H104, H105, H106, H107, H108, H109, H11, H110, H111, H112, H113, H114, H115, H116, H117, H118, H119, H12, H120, H121, H122, H123, H124, H125, H126, H127, H128, H129, H13, H130, H131, H132, H133, H134, H135, H136, H137, H138, H139, H14, H140, H141, H142, H143, H144, H145, H146, H147, H148, H149, H15, H150, H151, H152, H153, H154, H155, H156, H157, H158, H159, H16, H160, H161, H162, H163, H164, H165, H166, H167, H168, H169, H17, H170, H171, H172, H173, H174, H175, H176, H177, H178, H179, H18, H180, H181, H182, H183, H184, H185, H186, H187, H188, H189, H19, H190, H191, H192, H193, H194, H195, H196, H197, H198, H199, H2, H20, H200, H201, H202, H203, H204, H205, H206, H207, H208, H209, H21, H210, H211, H212, H213, H214, H215, H216, H217, H218, H219, H220, H221, H222, H223, H224, H225, H226, H227, H27, H28, H29, H3, H30, H31, H4, H5, H53, H54, H55, H56, H57, H58, H59, H6, H60, H61, H62, H63, H64, H65, H66, H67, H68, H69, H7, H70, H71, H72, H73, H74, H75, H76, H77, H78, H79, H8, H80, H81, H82, H83, H84, H85, H86, H87, H88, H89, H9, H90, H91, H92, H93, H94, H95, H96, H97, H98, H99: MOUNT-HOLE2.8, holes:2,8
- moved H32 458.9 mm to (4.35, 410.4)
- moved H33 458.9 mm to (67.3, 410.4)
- moved H34 458.9 mm to (67.3, 440.4)
- moved H45 449.0 mm to (4.35, 60.2), turned to 180 degrees
- moved H43 438.0 mm to (4.35, 117.3)
- moved H36 432.2 mm to (67.3, 448.4)
- moved H35 432.2 mm to (4.35, 448.4)
- moved H47 384.8 mm to (4.35, 3.25), turned to 180 degrees
- moved H48 363.3 mm to (4.35, 125.3)
- moved H51 322.8 mm to (4.35, 212.3)
- moved H52 322.8 mm to (67.3, 212.3)
- moved H44 313.4 mm to (67.3, 117.3)
- moved H42 308.0 mm to (67.3, 60.4)
- moved H50 298.7 mm to (67.3, 155.3)
- moved H25 286.1 mm to (4.35, 402.4)
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Other:
- board size 702.4 x 426.4 mm -> 103.1 x 451.4 mm
