File: case/gameboyzero.brd (EAGLE design)
At the start: 103.1 x 451.4 mm, 26 parts

Commit message: Tue Nov  7 23:54:05 EST 2017
Parts:
- added H1, H10, H100, H101, H102, H103, H104, H105, H106, H107, H108, H109, H11, H110, H111, H112, H113, H114, H115, H116, H117, H118, H119, H12, H120, H121, H122, H123, H124, H125, H126, H127, H128, H129, H13, H130, H131, H132, H133, H134, H135, H136, H137, H138, H139, H14, H140, H141, H142, H143, H144, H145, H146, H147, H148, H149, H15, H150, H151, H152, H153, H154, H155, H156, H157, H158, H159, H16, H160, H161, H162, H163, H164, H165, H166, H167, H168, H169, H17, H170, H171, H172, H173, H174, H175, H176, H177, H178, H179, H18, H180, H181, H182, H183, H184, H185, H186, H187, H188, H189, H19, H190, H191, H192, H193, H194, H195, H196, H197, H198, H199, H2, H20, H200, H201, H202, H203, H204, H205, H206, H207, H208, H21, H27, H28, H29, H3, H30, H31, H4, H5, H53, H54, H55, H56, H57, H58, H59, H6, H60, H61, H62, H63, H64, H65, H66, H67, H68, H69, H7, H70, H71, H72, H73, H74, H75, H76, H77, H78, H79, H8, H80, H81, H82, H83, H84, H85, H86, H87, H88, H89, H9, H90, H91, H92, H93, H94, H95, H96, H97, H98, H99: MOUNT-HOLE2.8, holes:2,8
- moved H35 5.00 mm to (4.35, 443.4)
- moved H36 5.00 mm to (67.3, 443.4)
- moved H32 4.00 mm to (4.35, 406.4)
- moved H33 4.00 mm to (67.3, 406.4)
- moved H34 4.00 mm to (67.3, 436.4)
- moved H22 3.00 mm to (4.35, 312.4)
- moved H23 3.00 mm to (67.3, 312.4)
- moved H24 3.00 mm to (67.3, 342.4)
- moved H25 3.00 mm to (4.35, 399.4)
- moved H26 3.00 mm to (67.3, 399.4)
- moved H37 2.00 mm to (4.35, 218.3)
- moved H38 2.00 mm to (67.3, 218.3)
- moved H39 2.00 mm to (67.3, 248.3)
- moved H40 2.00 mm to (4.35, 305.4)
- moved H41 2.00 mm to (67.3, 305.4)
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Other:
- board size 103.1 x 451.4 mm -> 675.1 x 446.4 mm

Commit message: Tue Nov  7 23:58:46 EST 2017
Parts:
- moved H1 3.61 mm to (78.3, 314.4)
- moved H10 3.61 mm to (141.3, 445.4)
- moved H100 3.61 mm to (220.3, 126.3)
- moved H101 3.61 mm to (283.4, 126.3)
- moved H102 3.61 mm to (283.4, 156.3)
- moved H103 3.61 mm to (220.3, 213.3)
- moved H104 3.61 mm to (283.4, 213.3)
- moved H105 3.61 mm to (291.4, 314.4)
- moved H106 3.61 mm to (354.4, 314.4)
- moved H107 3.61 mm to (354.4, 344.4)
- moved H108 3.61 mm to (291.4, 401.4)
- moved H109 3.61 mm to (354.4, 401.4)
- moved H11 3.61 mm to (78.3, 220.3)
- moved H110 3.61 mm to (291.4, 408.4)
- moved H111 3.61 mm to (354.4, 408.4)
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Other:
- board size 675.1 x 446.4 mm -> 675.1 x 448.4 mm

Commit message: Wed  8 Nov 2017 12:24:01 EST
Parts:
- added H209, H210, H211, H212, H213, H214, H215, H216, H217, H218, H219, H220, H221, H222, H223, H224, H225, H226, H227, H228, H229, H230, H231, H232, H233, H234, H235, H236, H237, H238, H239, H240, H241, H242, H243, H244, H245, H246, H247, H248, H249, H250, H251, H252, H253, H254, H255, H256, H257, H258, H259, H260, H261, H262, H263, H264, H265, H266, H267, H268, H269, H270, H271, H272, H273, H274, H275, H276, H277, H278, H279, H280, H281, H282, H283, H284, H285, H286, H287, H288, H289, H290, H291, H292, H293, H294, H295, H296, H297, H298, H299, H300, H301, H302, H303, H304, H305, H306: MOUNT-HOLE2.8, holes:2,8
- moved H150 746.3 mm to (150.0, 700.0), turned to 0 degrees
- moved H98 717.7 mm to (78.0, 694.0)
- moved H151 709.5 mm to (213.0, 700.0), turned to 0 degrees
- moved H99 708.1 mm to (78.0, 700.0), turned to 0 degrees
- moved H204 705.5 mm to (222.0, 706.0)
- moved H20 695.0 mm to (6.00, 688.0), turned to 0 degrees
- moved H146 683.6 mm to (150.0, 688.0)
- moved H180 683.0 mm to (222.0, 545.0), turned to 0 degrees
- moved H196 682.2 mm to (222.0, 682.0)
- moved H21 681.7 mm to (69.0, 688.0), turned to 0 degrees
- moved H149 665.4 mm to (150.0, 694.0)
- moved H199 659.6 mm to (285.0, 694.0)
- moved H200 659.6 mm to (222.0, 694.0)
- moved H94 652.8 mm to (78.0, 682.0), turned to 180 degrees
- moved H197 650.6 mm to (222.0, 688.0), turned to 0 degrees
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Other:
- board size 675.1 x 448.4 mm -> 465.4 x 709 mm

Commit message: Mon 20 Nov 2017 21:17:25 EST
Parts:
- removed H1, H10, H11, H12, H13, H14, H15, H158, H159, H160, H2, H232, H233, H234, H235, H236, H237, H238, H239, H240, H241, H242, H243, H244, H245, H246, H247, H248, H249, H250, H251, H252, H253, H254, H255, H256, H257, H258, H259, H260, H261, H262, H263, H264, H265, H266, H267, H268, H269, H27, H270, H271, H272, H273, H274, H275, H276, H277, H278, H279, H28, H280, H281, H282, H283, H284, H285, H286, H287, H288, H289, H29, H290, H291, H292, H293, H294, H295, H296, H297, H298, H299, H3, H30, H300, H301, H302, H303, H304, H305, H306, H31, H4, H5, H6, H7, H8, H9: MOUNT-HOLE2.8, holes:2,8
- moved H150 721.1 mm to (357.3, 9.34), turned to 180 degrees
- moved H98 698.3 mm to (215.3, 9.34)
- moved H151 695.4 mm to (294.3, 9.34), turned to 180 degrees
- moved H99 694.6 mm to (152.3, 9.34), turned to 180 degrees
- moved H224 672.9 mm to (204.4, 660.3), turned to 90 degrees
- moved H146 656.3 mm to (357.3, 65.3)
- moved H149 644.0 mm to (294.3, 66.3)
- moved H220 639.2 mm to (9.36, 597.3), turned to 90 degrees
- moved H94 631.8 mm to (215.3, 65.3), turned to 0 degrees
- moved H97 627.8 mm to (152.3, 66.3)
- moved H153 612.8 mm to (357.3, 129.3), turned to 0 degrees
- moved H221 612.5 mm to (9.36, 660.3), turned to 90 degrees
- moved H225 610.2 mm to (147.4, 597.3), turned to 90 degrees
- moved H223 601.3 mm to (234.4, 660.3), turned to 90 degrees
- moved H148 589.6 mm to (357.3, 122.3), turned to 0 degrees
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Other:
- board size 465.4 x 709 mm -> 458.1 x 664.3 mm
