File: eagle/gameboyzero.sch (EAGLE design)
At the start: 22 parts

Commit message: Fri 13 Oct 2017 16:15:10 EDT
Parts:
- added H1: MOUNT-HOLE2.8, holes:MOUNT-HOLE2.8
Changed lines of the file:
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@@
 <part name="GND26" library="supply1" library_urn="urn:adsk.eagle:library:371" deviceset="GND" device=""/>
 <part name="GND27" library="supply1" library_urn="urn:adsk.eagle:library:371" deviceset="GND" device=""/>
+<part name="H1" library="holes" library_urn="urn:adsk.eagle:library:237" deviceset="MOUNT-HOLE" device="2.8" package3d_urn="urn:adsk.eagle:package:14271/1"/>
 </parts>
 <sheets>
@@
 <instance part="GND26" gate="1" x="48.26" y="57.658" rot="R270"/>
 <instance part="GND27" gate="1" x="226.06" y="78.74" rot="R90"/>
+<instance part="H1" gate="G$1" x="127" y="134.62"/>
 </instances>
 <busses>
