File: eagle/gameboyzero/gameboyzero.brd (EAGLE design)
At the start: 71 x 94 mm, 27 parts

Commit message: last minute fixes before production
Connections:
- net LEFT: now also PI1.15, PI1.55; no longer PI1.40, PI1.80
Routing:
- net LEFT: track 95.9 -> 75.8 mm
Changed lines of the file:
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@@
 <setting verticaltext="up"/>
 </settings>
-<grid distance="0.086" unitdist="mm" unit="mm" style="lines" multiple="1" display="yes" altdistance="0.25" altunitdist="mm" altunit="mm"/>
+<grid distance="1" unitdist="mm" unit="mm" style="lines" multiple="1" display="yes" altdistance="0.25" altunitdist="mm" altunit="mm"/>
 <layers>
 <layer number="1" name="Top" color="4" fill="1" visible="yes" active="yes"/>
 <layer number="2" name="Route2" color="1" fill="3" visible="no" active="yes"/>
 <layer number="15" name="Route15" color="4" fill="6" visible="no" active="yes"/>
-<layer number="16" name="Bottom" color="1" fill="1" visible="no" active="yes"/>
+<layer number="16" name="Bottom" color="1" fill="1" visible="yes" active="yes"/>
 <layer number="17" name="Pads" color="2" fill="1" visible="yes" active="yes"/>
 <layer number="18" name="Vias" color="2" fill="1" visible="yes" active="yes"/>
@@
 <layer number="20" name="Dimension" color="15" fill="1" visible="yes" active="yes"/>
 <layer number="21" name="tPlace" color="7" fill="1" visible="yes" active="yes"/>
-<layer number="22" name="bPlace" color="7" fill="1" visible="no" active="yes"/>
+<layer number="22" name="bPlace" color="7" fill="1" visible="yes" active="yes"/>
 <layer number="23" name="tOrigins" color="15" fill="1" visible="yes" active="yes"/>
-<layer number="24" name="bOrigins" color="15" fill="1" visible="no" active="yes"/>
+<layer number="24" name="bOrigins" color="15" fill="1" visible="yes" active="yes"/>
 <layer number="25" name="tNames" color="7" fill="1" visible="yes" active="yes"/>
-<layer number="26" name="bNames" color="7" fill="1" visible="no" active="yes"/>
+<layer number="26" name="bNames" color="7" fill="1" visible="yes" active="yes"/>
 <layer number="27" name="tValues" color="7" fill="1" visible="yes" active="yes"/>
-<layer number="28" name="bValues" color="7" fill="1" visible="no" active="yes"/>
+<layer number="28" name="bValues" color="7" fill="1" visible="yes" active="yes"/>
 <layer number="29" name="tStop" color="7" fill="3" visible="no" active="yes"/>
 <layer number="30" name="bStop" color="7" fill="6" visible="no" active="yes"/>
@@
 <vertex x="0" y="94"/>
 </polygon>
-<via x="12" y="55" extent="1-16" drill="0.5"/>
+<via x="9" y="55" extent="1-16" drill="0.5"/>
 <via x="39" y="83" extent="1-16" drill="0.5"/>
 <via x="40" y="70" extent="1-16" drill="0.5"/>
@@
 </signal>
 <signal name="LEFT">
-<contactref element="PI1" pad="40"/>
 <contactref element="BTN_LEFT" pad="B2"/>
-<wire x1="57.087" y1="59" x2="57.087" y2="44" width="0.3048" layer="16"/>
-<wire x1="3.598259375" y1="18.21975625" x2="3.623259375" y2="24.1" width="0.3048" layer="1"/>
-<wire x1="27" y1="26.5" x2="27" y2="44" width="0.3048" layer="1"/>
-<wire x1="27" y1="44" x2="57.087" y2="44" width="0.3048" layer="1"/>
-<via x="57.087" y="44" extent="1-16" drill="0.5"/>
-<wire x1="3.623259375" y1="24.1" x2="17.5" y2="24.1" width="0.3048" layer="1"/>
-<wire x1="17.5" y1="24.1" x2="17.5" y2="26.5" width="0.3048" layer="1"/>
-<wire x1="17.5" y1="26.5" x2="27" y2="26.5" width="0.3048" layer="1"/>
-<contactref element="PI1" pad="80"/>
-<wire x1="57.087" y1="60.457" x2="57.087" y2="59" width="0.254" layer="16"/>
-<wire x1="57.087" y1="58.806" x2="57.087" y2="59" width="0.4064" layer="16"/>
+<contactref element="PI1" pad="55"/>
+<contactref element="PI1" pad="15"/>
+<wire x1="3.598259375" y1="18.21975625" x2="3.598259375" y2="28" width="0.3048" layer="1"/>
+<wire x1="3.598259375" y1="28" x2="10" y2="28" width="0.3048" layer="1"/>
+<wire x1="10" y1="28" x2="10" y2="49" width="0.3048" layer="1"/>
+<wire x1="10" y1="49" x2="12.6" y2="49" width="0.3048" layer="1"/>
+<via x="12.6" y="53" extent="1-16" drill="0.5"/>
+<wire x1="12.6" y1="53" x2="12.6" y2="67" width="0.3048" layer="16"/>
+<wire x1="12.6" y1="67" x2="26.607" y2="67" width="0.3048" layer="16"/>
+<wire x1="26.607" y1="64.648" x2="26.607" y2="67" width="0.3048" layer="16"/>
+<wire x1="12.6" y1="49" x2="12.6" y2="53" width="0.3048" layer="1"/>
+<wire x1="26.607" y1="64.648" x2="26.607" y2="62.997" width="0.3048" layer="16"/>
 </signal>
 <signal name="DOWN">
