File: eagle/gameboyzero-split-board/gameboyzero-split-top.brd (EAGLE design)
At the start: 142 x 94 mm, 36 parts

Commit message: Mon 27 Nov 2017 11:39:46 EST
Parts:
- removed BTN_L1, BTN_L2, BTN_R1, BTN_R2: MOMENTARY-SWITCH-SPST-SMD-12MM, SparkFun-Switches:TACTILE_SWITCH_SMD_12MM
- removed H10, H6, H7, H8, H9: MOUNT-HOLE2.8, holes:3,0
- removed J3: (no value), SparkFun-Connectors:1X06
- removed LED2: (no value), adafruit:CHIPLED_0805
- removed R3: 1K, adafruit:R0805
Connections:
- removed net LED1: LED2.A, R3.1
- net GND: no longer BTN_L1.1, BTN_L2.1, BTN_R1.1, BTN_R2.1, J3.1, LED2.C
- net L1: no longer BTN_L1.3, J3.5
- net L2: no longer BTN_L2.3, J3.4
- net R1: no longer BTN_R1.3, J3.2
- net R2: no longer BTN_R2.3, J3.3
- net SWITCH_OUT+: no longer J3.6, R3.2
Routing:
- net SWITCH_OUT+: track 212.6 -> 158.8 mm
- net LED1: track 25.2 -> 0.00 mm
- net L2: track 83.0 -> 58.9 mm
- net R2: track 78.5 -> 59.1 mm
- net L1: track 70.1 -> 56.9 mm
- net R1: track 82.6 -> 74.2 mm
Other:
- board size 142 x 94 mm -> 71 x 94 mm
