File: eagle/gameboyzero-split-board/gameboyzero-split-top.brd (EAGLE design)
At the start: 71 x 94 mm, 24 parts

Commit message: Wed  6 Dec 2017 14:49:20 EST
Parts:
- moved J2 32.6 mm to (37.0, 3.00)
Routing:
- net R2: track 59.1 -> 85.1 mm, vias 2 -> 0
- net L2: track 58.9 -> 76.9 mm, vias 3 -> 0
- net L1: track 56.9 -> 72.9 mm, vias 2 -> 1
- net R1: track 74.2 -> 84.2 mm
- net SWITCH_OUT+: track 158.8 -> 164.8 mm, vias 3 -> 2
Changed lines of the file:
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@@
 <layers>
 <layer number="1" name="Top" color="4" fill="1" visible="yes" active="yes"/>
-<layer number="2" name="Route2" color="1" fill="3" visible="no" active="yes"/>
-<layer number="15" name="Route15" color="4" fill="6" visible="no" active="yes"/>
-<layer number="16" name="Bottom" color="1" fill="1" visible="no" active="yes"/>
+<layer number="2" name="Route2" color="1" fill="3" visible="yes" active="yes"/>
+<layer number="15" name="Route15" color="4" fill="6" visible="yes" active="yes"/>
+<layer number="16" name="Bottom" color="1" fill="1" visible="yes" active="yes"/>
 <layer number="17" name="Pads" color="2" fill="1" visible="yes" active="yes"/>
 <layer number="18" name="Vias" color="2" fill="1" visible="yes" active="yes"/>
@@
 <layer number="20" name="Dimension" color="15" fill="1" visible="yes" active="yes"/>
 <layer number="21" name="tPlace" color="7" fill="1" visible="yes" active="yes"/>
-<layer number="22" name="bPlace" color="7" fill="1" visible="no" active="yes"/>
+<layer number="22" name="bPlace" color="7" fill="1" visible="yes" active="yes"/>
 <layer number="23" name="tOrigins" color="15" fill="1" visible="yes" active="yes"/>
-<layer number="24" name="bOrigins" color="15" fill="1" visible="no" active="yes"/>
+<layer number="24" name="bOrigins" color="15" fill="1" visible="yes" active="yes"/>
 <layer number="25" name="tNames" color="7" fill="1" visible="yes" active="yes"/>
-<layer number="26" name="bNames" color="7" fill="1" visible="no" active="yes"/>
-<layer number="27" name="tValues" color="7" fill="1" visible="no" active="yes"/>
-<layer number="28" name="bValues" color="7" fill="1" visible="no" active="yes"/>
+<layer number="26" name="bNames" color="7" fill="1" visible="yes" active="yes"/>
+<layer number="27" name="tValues" color="7" fill="1" visible="yes" active="yes"/>
+<layer number="28" name="bValues" color="7" fill="1" visible="yes" active="yes"/>
 <layer number="29" name="tStop" color="7" fill="3" visible="no" active="yes"/>
 <layer number="30" name="bStop" color="7" fill="6" visible="no" active="yes"/>
@@
 <layer number="38" name="bTest" color="7" fill="1" visible="no" active="yes"/>
 <layer number="39" name="tKeepout" color="4" fill="11" visible="yes" active="yes"/>
-<layer number="40" name="bKeepout" color="1" fill="11" visible="no" active="yes"/>
+<layer number="40" name="bKeepout" color="1" fill="11" visible="yes" active="yes"/>
 <layer number="41" name="tRestrict" color="4" fill="10" visible="yes" active="yes"/>
-<layer number="42" name="bRestrict" color="1" fill="10" visible="no" active="yes"/>
+<layer number="42" name="bRestrict" color="1" fill="10" visible="yes" active="yes"/>
 <layer number="43" name="vRestrict" color="2" fill="10" visible="no" active="yes"/>
-<layer number="44" name="Drills" color="7" fill="1" visible="no" active="yes"/>
+<layer number="44" name="Drills" color="7" fill="1" visible="yes" active="yes"/>
 <layer number="45" name="Holes" color="7" fill="1" visible="yes" active="yes"/>
 <layer number="46" name="Milling" color="3" fill="1" visible="no" active="yes"/>
@@
 <layer number="50" name="dxf" color="7" fill="1" visible="no" active="no"/>
 <layer number="51" name="tDocu" color="7" fill="1" visible="yes" active="yes"/>
-<layer number="52" name="bDocu" color="7" fill="1" visible="no" active="yes"/>
+<layer number="52" name="bDocu" color="7" fill="1" visible="yes" active="yes"/>
 <layer number="53" name="tGND_GNDA" color="7" fill="1" visible="no" active="no"/>
 <layer number="54" name="bGND_GNDA" color="7" fill="1" visible="no" active="no"/>
@@
 <attribute name="SF_ID" value="PRT-08612" x="34.654" y="47.902" size="1.778" layer="28" rot="MR90" display="off"/>
 </element>
-<element name="J2" library="SparkFun-Connectors" library_urn="urn:adsk.eagle:library:513" package="1X06" package3d_urn="urn:adsk.eagle:package:38009/1" value="" x="43" y="35" rot="R180">
-<attribute name="PROD_ID" value="CONN-08437" x="43" y="35" size="1.778" layer="27" rot="R180" display="off"/>
+<element name="J2" library="SparkFun-Connectors" library_urn="urn:adsk.eagle:library:513" package="1X06" package3d_urn="urn:adsk.eagle:package:38009/1" value="" x="37" y="3" rot="R180">
+<attribute name="PROD_ID" value="CONN-08437" x="37" y="3" size="1.778" layer="27" rot="R180" display="off"/>
 </element>
 </elements>
@@
 <contactref element="PI1" pad="20"/>
 <contactref element="J2" pad="1"/>
-<via x="33.5" y="10" extent="1-16" drill="0.5"/>
+<via x="40.5" y="36" extent="1-16" drill="0.5"/>
 </signal>
 <signal name="RESET">
@@
 <contactref element="BTN_DOWN" pad="B2"/>
 <wire x1="46.927" y1="59" x2="46.927" y2="43" width="0.3048" layer="16"/>
-<wire x1="13.780240625" y1="6.098259375" x2="25" y2="6.198259375" width="0.3048" layer="1"/>
-<wire x1="25" y1="6.198259375" x2="25" y2="25" width="0.3048" layer="1"/>
+<wire x1="13.780240625" y1="6.098259375" x2="25" y2="6.098259375" width="0.3048" layer="1"/>
+<wire x1="25" y1="6.098259375" x2="25" y2="25" width="0.3048" layer="1"/>
 <wire x1="25" y1="25" x2="26" y2="25" width="0.3048" layer="1"/>
 <wire x1="26" y1="25" x2="26" y2="43" width="0.3048" layer="1"/>
@@
 <wire x1="8.827" y1="59.568" x2="8.827" y2="58.806" width="0.254" layer="16"/>
 <contactref element="J2" pad="6"/>
-<wire x1="6" y1="25" x2="29" y2="25" width="0.6096" layer="16"/>
 <wire x1="6" y1="59.568" x2="6" y2="25" width="0.6096" layer="16"/>
-<wire x1="30.3" y1="35" x2="29" y2="35" width="0.6096" layer="1"/>
-<wire x1="29" y1="35" x2="29" y2="25" width="0.6096" layer="1"/>
-<via x="29" y="25" extent="1-16" drill="0.5"/>
+<wire x1="6" y1="25" x2="13" y2="25" width="0.6096" layer="16"/>
+<wire x1="13" y1="25" x2="13" y2="8" width="0.6096" layer="16"/>
+<wire x1="13" y1="8" x2="24.3" y2="8" width="0.6096" layer="16"/>
+<wire x1="24.3" y1="8" x2="24.3" y2="3" width="0.6096" layer="16"/>
 </signal>
 <signal name="BATT+">
@@
 <contactref element="J2" pad="5"/>
 <wire x1="21.527" y1="59.568" x2="21.527" y2="50" width="0.3048" layer="16"/>
-<wire x1="16" y1="50" x2="16" y2="30" width="0.3048" layer="16"/>
-<via x="16" y="30" extent="1-16" drill="0.5"/>
-<wire x1="16" y1="30" x2="20" y2="30" width="0.3048" layer="1"/>
-<via x="20" y="30" extent="1-16" drill="0.5"/>
-<wire x1="20" y1="30" x2="32.84" y2="30" width="0.3048" layer="16"/>
-<wire x1="32.84" y1="30" x2="32.84" y2="35" width="0.3048" layer="16"/>
 <wire x1="21.527" y1="50" x2="16" y2="50" width="0.3048" layer="16"/>
+<wire x1="16" y1="11" x2="26.84" y2="11" width="0.3048" layer="16"/>
+<wire x1="16" y1="50" x2="16" y2="11" width="0.3048" layer="16"/>
+<via x="26.84" y="11" extent="1-16" drill="0.5"/>
+<wire x1="26.84" y1="3" x2="26.84" y2="11" width="0.3048" layer="1"/>
 </signal>
 <signal name="L2">
@@
 <contactref element="J2" pad="4"/>
 <wire x1="18.987" y1="52" x2="18.987" y2="58.806" width="0.3048" layer="16"/>
-<wire x1="35.38" y1="35" x2="35.38" y2="31" width="0.3048" layer="1"/>
-<wire x1="35.38" y1="31" x2="31" y2="31" width="0.3048" layer="1"/>
-<via x="31" y="31" extent="1-16" drill="0.5"/>
-<wire x1="31" y1="31" x2="21" y2="31" width="0.3048" layer="16"/>
-<via x="21" y="31" extent="1-16" drill="0.5"/>
-<wire x1="21" y1="31" x2="14" y2="31" width="0.3048" layer="1"/>
-<via x="14" y="31" extent="1-16" drill="0.5"/>
-<wire x1="14" y1="31" x2="14" y2="52" width="0.3048" layer="16"/>
-<wire x1="14" y1="52" x2="18.987" y2="52" width="0.3048" layer="16"/>
+<wire x1="18.987" y1="52" x2="14" y2="52" width="0.3048" layer="16"/>
+<wire x1="29.38" y1="9" x2="14" y2="9" width="0.3048" layer="16"/>
+<wire x1="14" y1="52" x2="14" y2="9" width="0.3048" layer="16"/>
+<wire x1="29.38" y1="3" x2="29.38" y2="9" width="0.3048" layer="16"/>
 </signal>
 <signal name="R1">
@@
 <wire x1="22.75" y1="49" x2="18" y2="49" width="0.3048" layer="16"/>
 <wire x1="22.75" y1="63.886" x2="22.75" y2="49" width="0.3048" layer="16"/>
-<wire x1="18" y1="49" x2="18" y2="27" width="0.3048" layer="16"/>
-<wire x1="40.46" y1="27" x2="40.46" y2="35" width="0.3048" layer="16"/>
-<wire x1="18" y1="27" x2="40.46" y2="27" width="0.3048" layer="16"/>
+<wire x1="18" y1="49" x2="18" y2="15" width="0.3048" layer="16"/>
+<wire x1="18" y1="15" x2="34.46" y2="15" width="0.3048" layer="16"/>
+<wire x1="34.46" y1="15" x2="34.46" y2="3" width="0.3048" layer="16"/>
 </signal>
 <signal name="R2">
@@
 <wire x1="20.35" y1="63.886" x2="20.35" y2="51" width="0.3048" layer="16"/>
 <wire x1="20.35" y1="51" x2="15" y2="51" width="0.3048" layer="16"/>
-<wire x1="15" y1="51" x2="15" y2="38" width="0.3048" layer="16"/>
-<via x="15" y="38" extent="1-16" drill="0.5"/>
-<wire x1="15" y1="38" x2="22" y2="38" width="0.3048" layer="1"/>
-<via x="22" y="38" extent="1-16" drill="0.5"/>
-<wire x1="22" y1="38" x2="37.92" y2="38" width="0.3048" layer="16"/>
-<wire x1="37.92" y1="38" x2="37.92" y2="35" width="0.3048" layer="16"/>
+<wire x1="15" y1="51" x2="15" y2="10" width="0.3048" layer="16"/>
+<wire x1="31.92" y1="10" x2="31.92" y2="3" width="0.3048" layer="16"/>
+<wire x1="15" y1="10" x2="31.92" y2="10" width="0.3048" layer="16"/>
 </signal>
 <signal name="LED">
