File: eagle/gameboyzero-split-board/gameboyzero-split-bottom.brd (EAGLE design)
At the start: 71 x 94 mm, 12 parts

Commit message: Wed  6 Dec 2017 14:49:20 EST
Parts:
- moved J3 32.6 mm to (37.0, 3.00)
Routing:
- net R1: track 8.47 -> 41.1 mm
- net SWITCH_OUT+: track 53.8 -> 79.8 mm
- net L1: track 13.2 -> 24.8 mm
- net L2: track 24.1 -> 13.9 mm
- net R2: track 19.4 -> 24.4 mm
