File: case/gameboyzero-split-board/gameboyzero-split-board.brd (EAGLE design)
At the start: 460.3 x 677.4 mm, 240 parts

Commit message: Fri 12 Jan 2018 17:10:25 EST
Parts:
- removed H1, H10, H100, H101, H102, H103, H104, H105, H106, H107, H108, H109, H11, H110, H111, H112, H113, H114, H115, H116, H117, H118, H119, H12, H120, H121, H122, H123, H124, H125, H126, H127, H128, H129, H13, H130, H131, H132, H133, H134, H135, H136, H137, H138, H139, H14, H140, H141, H142, H143, H144, H145, H146, H147, H148, H149, H15, H150, H151, H152, H153, H154, H155, H156, H157, H158, H159, H16, H160, H161, H162, H163, H164, H165, H166, H167, H168, H169, H17, H170, H171, H172, H173, H174, H175, H176, H177, H178, H179, H18, H180, H181, H182, H183, H184, H185, H186, H187, H188, H189, H19, H190, H191, H192, H193, H194, H195, H196, H197, H198, H199, H2, H20, H200, H201, H202, H203, H204, H205, H206, H207, H208, H209, H21, H210, H211, H212, H213, H214, H215, H216, H217, H218, H219, H22, H220, H221, H222, H223, H224, H225, H226, H227, H228, H229, H23, H230, H231, H232, H233, H234, H235, H236, H237, H238, H239, H24, H240, H25, H26, H27, H28, H29, H3, H30, H31, H32, H33, H34, H35, H36, H37, H38, H39, H4, H40, H41, H42, H43, H44, H45, H46, H47, H48, H49, H5, H50, H51, H52, H53, H54, H55, H56, H57, H58, H59, H6, H60, H61, H62, H63, H64, H65, H66, H67, H68, H69, H7, H70, H71, H72, H73, H74, H75, H76, H77, H78, H79, H8, H80, H81, H82, H83, H84, H85, H86, H87, H88, H89, H9, H90, H91, H92, H93, H94, H95, H96, H97, H98, H99: MOUNT-HOLE2.8, holes:2,8
Other:
- board size 460.3 x 677.4 mm -> 402 x 244.7 mm

Commit message: simplified plexi
Other:
- board size 402 x 244.7 mm -> 118 x 244.7 mm
