File: case/gameboyzero-split-board/gameboyzero-split-board-single.brd (EAGLE design)
At the start: 355 x 464 mm, 0 parts

Commit message: Thu 22 Feb 2018 09:08:23 EST
Other:
- board size 355 x 464 mm -> 355 x 696 mm
